File: pcb/doorman.kicad_sch (KiCad schematic)
At the start: 45 parts, among them J1 USB_C_Receptacle_USB2.0, J2 Terminal, J3 3V3 Test Pad, J4 TX Test Pad, J5 RX Test Pad, J6 BUS Test Pad, J7 BUS RX Test Pad, Q1 BC817, SW1 Reset, SW2 Flash, U1 ESP32-S3-WROOM-1, U2 AP63203WU, U3 GAQY252G3S

Commit message: Fix PCB Files
Parts:
- removed C10, C11, C12, C9: 100nF, Capacitor_SMD:C_0603_1608Metric, symbol Device:C_Small
- removed C8: 33uF, symbol Device:C_Polarized
- removed R12: 10k, symbol Device:R
- added C8: 33uF, symbol Device:C_Polarized_Small
- C2: value 10uF -> 100nF
- C3: LCSC C2164331 -> C7471889; MPN EMZS350ARA471MHA0G -> 189RV0027; Package SMD,D8xL10mm -> SMD,D8xL10.5mm
- D1, D5, D6: LCSC C5451629 -> C191023
- D2: LCSC C3011144 -> C2886734
- D3: footprint LED_SMD:LED_WS2812B-2020_PLCC4_2.0x2.0mm -> Doorman:LED-SMD_4P-L2.0-W1.8_CY-0807; symbol LED:WS2812B-2020 -> easyeda2kicad:XL-0807RGBC-WS2812B; LCSC C965555 -> C41413181; LCSC Part (none) -> C3646929; MPN WS2812B-2020 -> XL-0807RGBC-WS2812B-S; Manufacturer_Name (none) -> XINGLIGHT; Manufacturer_Part_Number (none) -> XL-0807RGBC-WS2812B; Package SMD,2x2mm -> SMD,1.8x2mm
- D4: value Red LED -> Red
- J6: now fitted
- Q1: Height 1.1 -> (none); LCSC C39828 -> C5184412; MPN BC817-25,215 -> BC817-25; Manufacturer_Name NXP -> (none); Manufacturer_Part_Number BC817 -> (none); Mouser Part Number N/A -> (none); Mouser Price/Stock https://www.mouser.co.uk/ProductDetail/NXP-Semiconductors/B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 -> (none)
- R11: value 10k -> 10K; footprint (none) -> Resistor_SMD:R_0603_1608Metric; LCSC (none) -> C25804; MPN (none) -> 0603WAF1002T5E; Package (none) -> 0603; now not fitted
- R5: value 10K -> 1M; LCSC C25804 -> C22935; MPN 0603WAF1002T5E -> 0603WAF1004T5E
- R6: value 1.6K -> 147K; LCSC C25804 -> C22878; MPN 0603WAF1002T5E -> 0603WAF1473T5E
- R8: now not fitted
- SW1: value Reset -> Reset Button; LCSC C231329 -> C49234121; MPN B3U-1000P -> HX-B3U-1000P-1.6N
- SW2: value Flash -> Flash Button; LCSC C231329 -> C49234121; MPN B3U-1000P -> HX-B3U-1000P-1.6N
Connections:
- net +24V Bus: now also C8.1
- net +3.3V: now also D3.1 (VDD), J2.5 (Pin_5), R8.1; no longer D3.4 (VDD), R11.1
- net ADC_IN: now also R8.2, C8.2
- net GND: now also D3.3 (GND), R11.1; no longer D3.2 (VSS)
- net IO41: now also J2.7 (Pin_7); no longer R8.2
- net IO0 renamed FLASH
- net IO1 renamed LED_RED
- net IO10 renamed BUS_ANA
- net IO11: no longer names the net of U1.19 (IO11)
- net IO12: no longer names the net of U1.20 (IO12)
- net IO13: no longer names the net of U1.21 (IO13)
- net IO14: no longer names the net of U1.22 (IO14)
- net IO15: no longer names the net of U1.8 (IO15)
- net IO16: no longer names the net of U1.9 (IO16)
- net IO17: no longer names the net of U1.10 (IO17)
- net IO18: no longer names the net of U1.11 (IO18)
- net IO2 renamed LED_RGB
- net LED_RGB: now also D3.4 (DIN); no longer D3.3 (DIN)
- net IO21: no longer names the net of U1.23 (IO21)
- net IO38: no longer names the net of U1.31 (IO38)
- net IO42 renamed SSR
- net IO47: no longer names the net of U1.24 (IO47)
- net IO48: no longer names the net of U1.25 (IO48)
- net IO48: no longer J2.5 (Pin_5)
- net IO5: no longer names the net of U1.5 (IO5)
- net IO6: no longer names the net of U1.6 (IO6)
- net IO7: no longer names the net of U1.7 (IO7)
- net IO8 renamed BUS_TX
- net RX renamed RXD
- net TX renamed TXD
- no-connect marks 10 -> 25
Other:
- note added: "24VIN = ~3.0V 28VIN = ~3.6V"
- note added: "BUS AUDIO (TEST)"
- note added: "Capacitor needs to be directly connected to the bus. No Bridge rectifier inbetween!"
- note added: "No external ps"
- note removed: "~3.1V"
- moved on the sheet: C1, C2, C3, C4, C5, C6, C7, D1, D2, D4, D5, D6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

Commit message: Update pcb files
Connections:
- net at C3.1, C4.1, D1.1 (K)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: now also D6.1 (K); no longer R10.2
- net at R10.1: now also D6.2 (A); no longer D6.1 (K)
- net at JP1.1 (A): now also R10.2; no longer D6.2 (A)
- net IO4: no longer names the net of U1.4 (IO4)
- no-connect marks 25 -> 26
Other:
- moved on the sheet: C8, D1, D3, D4, D5, D6, JP1, R10, R11, R7, R8

Commit message: chore: Update pcb files
Parts:
- added JP2: SolderJumper_2_Open, Jumper:SolderJumper-2_P1.3mm_Open_RoundedPad1.0x1.5mm, symbol Jumper:SolderJumper_2_Open
- C8: footprint (none) -> Capacitor_SMD:C_1206_3216Metric_Pad1.33x1.80mm_HandSolder; now left out of the parts list
- R11, R8: footprint Resistor_SMD:R_0603_1608Metric -> Resistor_SMD:R_1206_3216Metric_Pad1.30x1.75mm_HandSolder; now left out of the parts list
Connections:
- net +24V Bus: no longer C8.1
- net ADC_IN: now also U1.7 (IO7)
- net BUS_WIRE1: now also JP2.1 (A)
- new net: C8.1, JP2.2 (B)
- no-connect marks 26 -> 25
Other:
- moved on the sheet: C8, R11, R8
