File: pcb/doorman.kicad_pcb (KiCad board)
At the start: 4 copper layers, 37.1 x 37.2 mm, 46 parts, among them J1 USB_C_Receptacle_USB2.0, J2 Terminal, J3 3V3 Test Pad, J4 TX Test Pad, J5 RX Test Pad, J6 BUS Test Pad, J7 BUS RX Test Pad, Q1 BC817, SW1 Reset, SW2 Flash, U1 ESP32-S3-WROOM-1, U2 AP63203WU, U3 GAQY252G3S

Commit message: Misc PCB
Parts:
- removed C8: 100nF, Capacitor_SMD:C_0603_1608Metric
- moved D1 0.32 mm to (138.4, 104.2)
Routing:
- net Net-(D6-A): track 11.6 -> 10.0 mm
- net +24V Bus: track 31.0 -> 30.4 mm
- net IO8: track 14.2 -> 13.6 mm
- net GND: vias 99 -> 112

Commit message: Fix PCB Files
Parts:
- removed C10, C11, C12, C9: 100nF, Capacitor_SMD:C_0603_1608Metric
- removed R8: 10K, Resistor_SMD:R_0603_1608Metric
- C2: value 10uF -> 100nF
- D3: footprint LED_SMD:LED_WS2812B-2020_PLCC4_2.0x2.0mm -> Doorman:LED-SMD_4P-L2.0-W1.8_CY-0807
- R5: value 10K -> 1M
- R6: value 1.6K -> 147K
- SW1: value Reset -> Reset Button
- SW2: value Flash -> Flash Button
- moved JP1 9.72 mm to (131.1, 100.2)
- moved D6 5.51 mm to (129.7, 98.0), turned to 0 degrees
- moved J3 3.20 mm to (129.7, 90.6)
- moved R10 2.99 mm to (128.4, 101.3), turned to -90 degrees
- moved R2 1.97 mm to (138.1, 111.8), turned to 0 degrees
- moved Q1 1.65 mm to (138.3, 109.1)
- moved D1 0.66 mm to (138.2, 104.8)
- moved C5 0.21 mm to (128.2, 92.9)
- moved C6 0.21 mm to (134.2, 89.5)
- moved C7 0.21 mm to (132.8, 89.5)
- moved C4 0.21 mm to (133.7, 94.2)
- moved L1 0.21 mm to (129.8, 88.9)
- moved U2 0.21 mm to (130.7, 93.8)
- moved C1 0.18 mm to (130.3, 84.0)
- moved R1 0.11 mm to (128.1, 84.8)
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Connections:
- net /IO0 renamed /FLASH
- net IO1 renamed LED_RED
- net IO10 renamed BUS_ANA
- net IO42 renamed SSR
- net IO8 renamed BUS_TX
- net RX renamed /RXD
- net TX renamed /TXD
- D3 pad 1: unconnected-(D3-DOUT-Pad1) -> +3.3V
- D3 pad 2: GND -> unconnected-(D3-DOUT-Pad2)
- D3 pad 3: IO2 -> GND
- D3 pad 4: +3.3V -> LED_RGB
- J2 pad 5: IO48 -> +3.3V
- J2 pad 7: Net-(J2-Pin_7) -> IO41
- U1 pad 10: IO17 -> unconnected-(U1-IO17-Pad10)
- U1 pad 11: IO18 -> unconnected-(U1-IO18-Pad11)
- U1 pad 19: IO11 -> unconnected-(U1-IO11-Pad19)
- U1 pad 20: IO12 -> unconnected-(U1-IO12-Pad20)
- U1 pad 21: IO13 -> unconnected-(U1-IO13-Pad21)
- U1 pad 22: IO14 -> unconnected-(U1-IO14-Pad22)
- U1 pad 23: IO21 -> unconnected-(U1-IO21-Pad23)
- U1 pad 24: IO47 -> unconnected-(U1-IO47-Pad24)
- U1 pad 25: IO48 -> unconnected-(U1-IO48-Pad25)
- U1 pad 31: IO38 -> unconnected-(U1-IO38-Pad31)
- U1 pad 38: IO2 -> LED_RGB
- U1 pad 5: IO5 -> unconnected-(U1-IO5-Pad5)
- U1 pad 6: IO6 -> unconnected-(U1-IO6-Pad6)
- U1 pad 7: IO7 -> unconnected-(U1-IO7-Pad7)
- U1 pad 8: IO15 -> unconnected-(U1-IO15-Pad8)
- U1 pad 9: IO16 -> unconnected-(U1-IO16-Pad9)
Routing:
- net +3.3V: track 36.7 -> 63.1 mm, vias 8 -> 5
- net IO48: track 12.5 -> 0.00 mm, vias 1 -> 0
- net LED_RGB: track 0.00 -> 12.2 mm, vias 0 -> 2
- net IO2: track 12.2 -> 0.00 mm, vias 2 -> 0
- net +24V Bus: track 30.4 -> 39.5 mm, vias 1 -> 2
- net Net-(D6-A): track 10.0 -> 2.23 mm, vias 1 -> 0
- net GND: track 16.9 -> 9.96 mm, vias 112 -> 59
- net Net-(D1-K): track 58.4 -> 52.2 mm
- net IO41: track 2.19 -> 7.97 mm
- net Net-(J2-Pin_7): track 5.26 -> 0.00 mm
- net BUS_TX: track 13.6 -> 18.6 mm
- net IO40: track 11.4 -> 8.40 mm, vias 1 -> 0
- net BUS_ANA: track 21.7 -> 19.4 mm
- net USB_D+: track 18.5 -> 19.7 mm
- net USB_D-: track 18.2 -> 18.9 mm
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- removed copper zone on In1.Cu, net +3.3V
Other:
- board text added: "BUS PWR"
- board text added: "U41"
- board text removed: "BTN"
- board text removed: "BUS"
- board text removed: "I48"
- board text removed: "PWR"

Commit message: Update pcb files
Parts:
- moved D1 6.60 mm to (138.6, 111.4)
- moved R2 5.83 mm to (136.6, 106.1), turned to 90 degrees
- moved R10 3.75 mm to (130.0, 97.9), turned to 0 degrees
- moved D6 2.96 mm to (128.2, 100.7), turned to 90 degrees
- moved Q1 2.46 mm to (138.8, 106.7)
- moved R3 1.20 mm to (144.2, 104.7)
- moved R4 0.89 mm to (148.2, 104.7)
- moved JP1 0.84 mm to (131.9, 100.2)
- moved C2 0.14 mm to (135.0, 84.8)
- moved R1 0.10 mm to (128.1, 84.7)
- moved C5 0.10 mm to (128.2, 92.8)
- moved C4 0.08 mm to (133.7, 94.2)
- moved C1 0.06 mm to (130.3, 83.9)
Connections:
- D6 pad 1: Net-(D6-K) -> Net-(D1-K)
- JP1 pad 1: Net-(D6-A) -> Net-(JP1-A)
- R10 pad 1: Net-(D6-K) -> Net-(D6-A)
- R10 pad 2: Net-(D1-K) -> Net-(JP1-A)
- U1 pad 4: IO4 -> unconnected-(U1-IO4-Pad4)
Routing:
- net BUS_TX: track 18.6 -> 8.82 mm, vias 2 -> 0
- net +5V: track 12.0 -> 17.0 mm
- net GND: track 9.96 -> 5.86 mm, vias 59 -> 72
- net +24V Bus: track 39.5 -> 36.5 mm
- net SSR: track 12.2 -> 15.1 mm
- net /FLASH: track 31.7 -> 34.6 mm
- net Net-(JP1-A): track 0.00 -> 2.46 mm
- net Net-(D1-K): track 52.2 -> 54.7 mm
- net +3.3V: track 63.1 -> 65.3 mm
- net Net-(D6-K): track 1.88 -> 0.00 mm
- net /EN: track 14.7 -> 14.0 mm
Other:
- board text added: "I41"
- board text added: "SERIAL"
- board text removed: "U41"
- board text removed: "USB-C"
