File: pcb/doorman.kicad_pcb (KiCad board)
At the start: 4 copper layers, 37.1 x 37.2 mm, 40 parts, among them J1 USB_C_Receptacle_USB2.0, J2 Terminal, J3 3V3 Test Pad, J4 TX Test Pad, J5 RX Test Pad, J6 BUS Test Pad, J7 BUS RX Test Pad, Q1 BC817, SW1 Reset Button, SW2 Flash Button, U1 ESP32-S3-WROOM-1, U2 AP63203WU, U3 GAQY252G3S

Commit message: chore: Add pcb2blender labels to pcb
Other:
- board text added: "PCB3D_BR_doorman"
- board text added: "PCB3D_TL_doorman"
Changed lines of the file:
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@@
+		)
+	)
+	(gr_text "PCB3D_TL_doorman"
+		(at 125.56 75.23 0)
+		(layer "Dwgs.User")
+		(effects
+			(font
+				(size 1.5 1.5)
+				(thickness 0.3)
+				(bold yes)
+			)
+			(justify left bottom)
+		)
+	)
+	(gr_text "PCB3D_BR_doorman"
+		(at 165.11 115.29 0)
+		(layer "Dwgs.User")
+		(effects
+			(font
+				(size 1.5 1.5)
+				(thickness 0.3)
+				(bold yes)
+			)
+			(justify left bottom)
 		)
 	)

Commit message: chore: Update pcb files
Parts:
- added 11: 10K, Resistor_SMD:R_1206_3216Metric_Pad1.30x1.75mm_HandSolder, B.Cu at (139.5, 89.7)
- added 8: 10K, Resistor_SMD:R_1206_3216Metric_Pad1.30x1.75mm_HandSolder, B.Cu at (136.6, 89.7)
- added C8: 33uF, Capacitor_SMD:C_1206_3216Metric_Pad1.33x1.80mm_HandSolder, B.Cu at (144.4, 99.3)
- added JP2: SolderJumper_2_Open, Jumper:SolderJumper-2_P1.3mm_Open_RoundedPad1.0x1.5mm, B.Cu at (158.5, 102.8)
Connections:
- U1 pad 7: unconnected-(U1-IO7-Pad7) -> ADC_IN
Routing:
- net ADC_IN: track 0.00 -> 14.6 mm, vias 0 -> 1
- net Net-(JP2-B): track 0.00 -> 13.7 mm
- net +3.3V: track 65.3 -> 68.3 mm
- net BUS_WIRE1: track 13.1 -> 16.1 mm
- net GND: track 5.86 -> 5.89 mm, vias 72 -> 70
